Commit message: fixed directions of rotation

File: crs_f3_robot_description/urdf/f3.urdf (robot description, URDF)
Before this commit: robot crs_f3, 9 links, 8 joints
Links:
- link base_link: mass 1 -> 0.165
- link link_1: mass 1 -> 0.496
- link link_2: mass 1 -> 0.140
- link link_3: mass 1 -> 0.105
- link link_4: mass 1 -> 0.105
- link link_5: mass 1 -> 0.011
- link link_6: mass 1 -> 0.006
Joints:
- joint joint_a1: axis 0 0 -1 -> 0 0 1
- joint joint_a2: axis 0 1 0 -> 0 -1 0; limit lower=-0.7853981633974483 upper=2.356194490192345 effort=0 velocity=3.6651914291880923 -> lower=-2.356194490192345 upper=0.7853981633974483 effort=0 velocity=3.6651914291880923
- joint joint_a3: axis 0 1 0 -> 0 -1 0
- joint joint_a4: axis 0 0 -1 -> 0 0 1
- joint joint_a5: axis 0 1 0 -> 0 -1 0
- joint joint_a6: axis 0 0 -1 -> 0 0 1

File: crs_f3_robot_description/urdf/f3_macro.xacro (robot description, xacro)
@@ -149,5 +149,5 @@
       <parent link="${prefix}base_link"/>
       <child link="${prefix}link_1"/>
-      <axis xyz="0 0 -1"/>
+      <axis xyz="0 0 1"/>
       <limit lower="${radians(-180)}" upper="${radians(180)}" effort="0" velocity="${radians(240)}"/>
     </joint>
@@ -156,6 +156,6 @@
       <parent link="${prefix}link_1"/>
       <child link="${prefix}link_2"/>
-      <axis xyz="0 1 0"/>
-      <limit lower="${radians(-45)}" upper="${radians(135)}" effort="0" velocity="${radians(210)}"/>
+      <axis xyz="0 -1 0"/>
+      <limit lower="${radians(-135)}" upper="${radians(45)}" effort="0" velocity="${radians(210)}"/>
     </joint>
     <joint name="${prefix}joint_a3" type="revolute">
@@ -163,5 +163,5 @@
       <parent link="${prefix}link_2"/>
       <child link="${prefix}link_3"/>
-      <axis xyz="0 1 0"/>
+      <axis xyz="0 -1 0"/>
       <limit lower="${radians(-135)}" upper="${radians(135)}" effort="0" velocity="${radians(240)}"/>
     </joint>
@@ -170,5 +170,5 @@
       <parent link="${prefix}link_3"/>
       <child link="${prefix}link_4"/>
-      <axis xyz="0 0 -1"/>
+      <axis xyz="0 0 1"/>
       <limit lower="${radians(-180)}" upper="${radians(180)}" effort="0" velocity="${radians(375)}"/>
     </joint>
@@ -177,5 +177,5 @@
       <parent link="${prefix}link_4"/>
       <child link="${prefix}link_5"/>
-      <axis xyz="0 1 0"/>
+      <axis xyz="0 -1 0"/>
       <limit lower="${radians(-135)}" upper="${radians(135)}" effort="0" velocity="${radians(300)}"/>
     </joint>
@@ -184,5 +184,5 @@
       <parent link="${prefix}link_5"/>
       <child link="${prefix}link_6"/>
-      <axis xyz="0 0 -1"/>
+      <axis xyz="0 0 1"/>
       <limit lower="${radians(-350)}" upper="${radians(350)}" effort="0" velocity="${radians(375)}"/>
     </joint>
