Commit message: latest model

File: crs_f3_robot_description/urdf/f3_macro.xacro (robot description, xacro)
@@ -18,6 +18,6 @@
       </collision>
       <inertial>
-        <origin xyz="0 0 -0.087" rpy="0 0 0"/>
-        <mass value="1"/>
+        <origin xyz="0 0 0.078" rpy="0 0 0"/>
+        <mass value="0.165"/>
         <inertia ixx="1.0" ixy="0.0" ixz="0.0" iyy="1.0" iyz="0.0" izz="1.0"/>
       </inertial>
@@ -38,6 +38,6 @@
       </collision>
       <inertial>
-        <origin xyz="${-0.1/2} ${-0.1/2} ${-0.350/2}" rpy="0 0 0"/>
-        <mass value="1"/>
+        <origin xyz="-0.014	-0.016	-0.133" rpy="0 0 0"/>
+        <mass value="0.496"/>
         <inertia ixx="1.0" ixy="0.0" ixz="0.0" iyy="1.0" iyz="0.0" izz="1.0"/>
       </inertial>
@@ -45,19 +45,19 @@
     <link name="${prefix}link_2">
       <visual>
+        <origin xyz="-0.1 -0.1 -0.350  " rpy="0 0 0" />
+        <geometry>
+          <mesh filename="package://crs_f3_robot_description/meshes/f3/visual/link_2.stl" />
+        </geometry>
+        <xacro:material_crs_ral_pure_white />
+      </visual>
+      <collision>
         <origin xyz="-0.1 -0.1 -0.350" rpy="0 0 0" />
         <geometry>
-          <mesh filename="package://crs_f3_robot_description/meshes/f3/visual/link_2.stl" />
-        </geometry>
-        <xacro:material_crs_ral_pure_white />
-      </visual>
-      <collision>
-        <origin xyz="-0.1 -0.1 -0.350" rpy="0 0 0" />
-        <geometry>
           <mesh filename="package://crs_f3_robot_description/meshes/f3/collision/link_2.stl" />
         </geometry>
       </collision>
       <inertial>
-        <origin xyz="${-0.1/2} ${-0.1/2} ${-0.615/2}" rpy="0 0 0"/>
-        <mass value="1"/>
+        <origin xyz="0 0 0" rpy="0 0 0"/>
+        <mass value="0.140"/>
         <inertia ixx="1.0" ixy="0.0" ixz="0.0" iyy="1.0" iyz="0.0" izz="1.0"/>
       </inertial>
@@ -72,5 +72,5 @@
       </visual>
       <collision>
-        <origin xyz="-0.1 -0.1 -0.615" rpy="0 0 0" />
+        <origin xyz="0	0.106	0.034" rpy="0 0 0" />
         <geometry>
           <mesh filename="package://crs_f3_robot_description/meshes/f3/collision/link_3.stl" />
@@ -78,6 +78,6 @@
       </collision>
       <inertial>
-        <origin xyz="${-0.1/2} ${0} ${-0.660/2}" rpy="0 0 0"/>
-        <mass value="1"/>
+        <origin xyz="0	0	0.112" rpy="0 0 0"/>
+        <mass value="0.105"/>
         <inertia ixx="1.0" ixy="0.0" ixz="0.0" iyy="1.0" iyz="0.0" izz="1.0"/>
       </inertial>
@@ -98,6 +98,6 @@
       </collision>
       <inertial>
-        <origin xyz="${-0.1/2} ${0} ${-0.885/2}" rpy="0 0 0"/>
-        <mass value="1"/>
+        <origin xyz="0	0	-0.112" rpy="0 0 0"/>
+        <mass value="0.105"/>
         <inertia ixx="1.0" ixy="0.0" ixz="0.0" iyy="1.0" iyz="0.0" izz="1.0"/>
       </inertial>
@@ -118,6 +118,6 @@
       </collision>
       <inertial>
-        <origin xyz="${-0.1/2} ${0} ${-0.960/2}" rpy="0 0 0"/>
-        <mass value="1"/>
+        <origin xyz="0	0	0.017" rpy="0 0 0"/>
+        <mass value="0.011"/>
         <inertia ixx="1.0" ixy="0.0" ixz="0.0" iyy="1.0" iyz="0.0" izz="1.0"/>
       </inertial>
@@ -138,6 +138,6 @@
       </collision>
       <inertial>
-        <origin xyz="${-0.1/2} ${0} ${-0.960}" rpy="0 0 0"/>
-        <mass value="1"/>
+        <origin xyz="0.1	0	0.88" rpy="0 0 0"/>
+        <mass value="0.006"/>
         <inertia ixx="1.0" ixy="0.0" ixz="0.0" iyy="1.0" iyz="0.0" izz="1.0"/>
       </inertial>
@@ -192,4 +192,67 @@
       <origin xyz="0 0 0" rpy="0 ${radians(90)} 0"/>
     </joint>
+    <transmission name="tran1">
+      <type>transmission_interface/SimpleTransmission</type>
+      <joint name="${prefix}joint_a1">
+        <hardwareInterface>hardware_interface/PositionJointInterface</hardwareInterface>
+      </joint>
+      <actuator name="motor1">
+        <hardwareInterface>hardware_interface/PositionJointInterface</hardwareInterface>
+        <mechanicalReduction>1</mechanicalReduction>
+      </actuator>
+    </transmission>
+    <transmission name="tran2">
+      <type>transmission_interface/SimpleTransmission</type>
+      <joint name="${prefix}joint_a2">
+        <hardwareInterface>hardware_interface/PositionJointInterface</hardwareInterface>
+      </joint>
+      <actuator name="motor2">
+        <hardwareInterface>hardware_interface/PositionJointInterface</hardwareInterface>
+        <mechanicalReduction>1</mechanicalReduction>
+      </actuator>
+    </transmission>
+    <transmission name="tran3">
+      <type>transmission_interface/SimpleTransmission</type>
+      <joint name="${prefix}joint_a3">
+        <hardwareInterface>hardware_interface/PositionJointInterface</hardwareInterface>
+      </joint>
+      <actuator name="motor3">
+        <hardwareInterface>hardware_interface/PositionJointInterface</hardwareInterface>
+        <mechanicalReduction>1</mechanicalReduction>
+      </actuator>
+    </transmission>
+    <transmission name="tran4">
+      <type>transmission_interface/SimpleTransmission</type>
+      <joint name="${prefix}joint_a4">
+        <hardwareInterface>hardware_interface/PositionJointInterface</hardwareInterface>
+      </joint>
+      <actuator name="motor4">
+        <hardwareInterface>hardware_interface/PositionJointInterface</hardwareInterface>
+        <mechanicalReduction>1</mechanicalReduction>
+      </actuator>
+    </transmission>
+    <transmission name="tran5">
+      <type>transmission_interface/SimpleTransmission</type>
+      <joint name="${prefix}joint_a5">
+        <hardwareInterface>hardware_interface/PositionJointInterface</hardwareInterface>
+      </joint>
+      <actuator name="motor5">
+        <hardwareInterface>hardware_interface/PositionJointInterface</hardwareInterface>
+        <mechanicalReduction>1</mechanicalReduction>
+      </actuator>
+    </transmission>
+    <transmission name="tran6">
+      <type>transmission_interface/SimpleTransmission</type>
+      <joint name="${prefix}joint_a6">
+        <hardwareInterface>hardware_interface/PositionJointInterface</hardwareInterface>
+      </joint>
+      <actuator name="motor6">
+        <hardwareInterface>hardware_interface/PositionJointInterface</hardwareInterface>
+        <mechanicalReduction>1</mechanicalReduction>
+      </actuator>
+    </transmission>
+    <gazebo>
+      <plugin name="control" filename="libgazebo_ros_control.so"/>
+    </gazebo>
     <!-- ROS base_link to crs $ROBROOT coordinate system transform -->
     <link name="world" />

Commit message: moveitconfig

File: crs_f3_robot_description/urdf/f3_macro.xacro (robot description, xacro)
@@ -192,66 +192,68 @@
       <origin xyz="0 0 0" rpy="0 ${radians(90)} 0"/>
     </joint>
-    <transmission name="tran1">
-      <type>transmission_interface/SimpleTransmission</type>
-      <joint name="${prefix}joint_a1">
-        <hardwareInterface>hardware_interface/PositionJointInterface</hardwareInterface>
-      </joint>
-      <actuator name="motor1">
-        <hardwareInterface>hardware_interface/PositionJointInterface</hardwareInterface>
-        <mechanicalReduction>1</mechanicalReduction>
-      </actuator>
-    </transmission>
-    <transmission name="tran2">
-      <type>transmission_interface/SimpleTransmission</type>
-      <joint name="${prefix}joint_a2">
-        <hardwareInterface>hardware_interface/PositionJointInterface</hardwareInterface>
-      </joint>
-      <actuator name="motor2">
-        <hardwareInterface>hardware_interface/PositionJointInterface</hardwareInterface>
-        <mechanicalReduction>1</mechanicalReduction>
-      </actuator>
-    </transmission>
-    <transmission name="tran3">
-      <type>transmission_interface/SimpleTransmission</type>
-      <joint name="${prefix}joint_a3">
-        <hardwareInterface>hardware_interface/PositionJointInterface</hardwareInterface>
-      </joint>
-      <actuator name="motor3">
-        <hardwareInterface>hardware_interface/PositionJointInterface</hardwareInterface>
-        <mechanicalReduction>1</mechanicalReduction>
-      </actuator>
-    </transmission>
-    <transmission name="tran4">
-      <type>transmission_interface/SimpleTransmission</type>
-      <joint name="${prefix}joint_a4">
-        <hardwareInterface>hardware_interface/PositionJointInterface</hardwareInterface>
-      </joint>
-      <actuator name="motor4">
-        <hardwareInterface>hardware_interface/PositionJointInterface</hardwareInterface>
-        <mechanicalReduction>1</mechanicalReduction>
-      </actuator>
-    </transmission>
-    <transmission name="tran5">
-      <type>transmission_interface/SimpleTransmission</type>
-      <joint name="${prefix}joint_a5">
-        <hardwareInterface>hardware_interface/PositionJointInterface</hardwareInterface>
-      </joint>
-      <actuator name="motor5">
-        <hardwareInterface>hardware_interface/PositionJointInterface</hardwareInterface>
-        <mechanicalReduction>1</mechanicalReduction>
-      </actuator>
-    </transmission>
-    <transmission name="tran6">
-      <type>transmission_interface/SimpleTransmission</type>
-      <joint name="${prefix}joint_a6">
-        <hardwareInterface>hardware_interface/PositionJointInterface</hardwareInterface>
-      </joint>
-      <actuator name="motor6">
-        <hardwareInterface>hardware_interface/PositionJointInterface</hardwareInterface>
-        <mechanicalReduction>1</mechanicalReduction>
-      </actuator>
+    <transmission name="trans_joint_a1">
+        <type>transmission_interface/SimpleTransmission</type>
+        <joint name="joint_a1">
+            <hardwareInterface>hardware_interface/EffortJointInterface</hardwareInterface>
+        </joint>
+        <actuator name="joint_a1_motor">
+            <hardwareInterface>hardware_interface/EffortJointInterface</hardwareInterface>
+            <mechanicalReduction>1</mechanicalReduction>
+        </actuator>
+    </transmission>
+    <transmission name="trans_joint_a2">
+        <type>transmission_interface/SimpleTransmission</type>
+        <joint name="joint_a2">
+            <hardwareInterface>hardware_interface/EffortJointInterface</hardwareInterface>
+        </joint>
+        <actuator name="joint_a2_motor">
+            <hardwareInterface>hardware_interface/EffortJointInterface</hardwareInterface>
+            <mechanicalReduction>1</mechanicalReduction>
+        </actuator>
+    </transmission>
+    <transmission name="trans_joint_a3">
+        <type>transmission_interface/SimpleTransmission</type>
+        <joint name="joint_a3">
+            <hardwareInterface>hardware_interface/EffortJointInterface</hardwareInterface>
+        </joint>
+        <actuator name="joint_a3_motor">
+            <hardwareInterface>hardware_interface/EffortJointInterface</hardwareInterface>
+            <mechanicalReduction>1</mechanicalReduction>
+        </actuator>
+    </transmission>
+    <transmission name="trans_joint_a4">
+        <type>transmission_interface/SimpleTransmission</type>
+        <joint name="joint_a4">
+            <hardwareInterface>hardware_interface/EffortJointInterface</hardwareInterface>
+        </joint>
+        <actuator name="joint_a4_motor">
+            <hardwareInterface>hardware_interface/EffortJointInterface</hardwareInterface>
+            <mechanicalReduction>1</mechanicalReduction>
+        </actuator>
+    </transmission>
+    <transmission name="trans_joint_a5">
+        <type>transmission_interface/SimpleTransmission</type>
+        <joint name="joint_a5">
+            <hardwareInterface>hardware_interface/EffortJointInterface</hardwareInterface>
+        </joint>
+        <actuator name="joint_a5_motor">
+            <hardwareInterface>hardware_interface/EffortJointInterface</hardwareInterface>
+            <mechanicalReduction>1</mechanicalReduction>
+        </actuator>
+    </transmission>
+    <transmission name="trans_joint_a6">
+        <type>transmission_interface/SimpleTransmission</type>
+        <joint name="joint_a6">
+            <hardwareInterface>hardware_interface/EffortJointInterface</hardwareInterface>
+        </joint>
+        <actuator name="joint_a6_motor">
+            <hardwareInterface>hardware_interface/EffortJointInterface</hardwareInterface>
+            <mechanicalReduction>1</mechanicalReduction>
+        </actuator>
     </transmission>
     <gazebo>
-      <plugin name="control" filename="libgazebo_ros_control.so"/>
+        <plugin name="gazebo_ros_control" filename="libgazebo_ros_control.so">
+            <robotNamespace>/</robotNamespace>
+        </plugin>
     </gazebo>
     <!-- ROS base_link to crs $ROBROOT coordinate system transform -->
